Commit message: Working Robot with first Correct Inertias etc.

File: install/brokk_tracked_test/share/brokk_tracked_test/urdf/brokk170_control_v2.xacro (robot description, xacro)
@@ -1,6 +1,6 @@
 <?xml version="1.0"?>
-<robot name="brokkmodel_v1" xmlns:xacro="http://ros.org/wiki/xacro">
+<robot name="brokkmodel_v2" xmlns:xacro="http://ros.org/wiki/xacro">
     <gazebo>
-        <plugin name="diff_drive_vorne" filename="libgazebo_ros_diff_drive.so">
+        <plugin name="diff_drive" filename="libgazebo_ros_diff_drive.so">
             <!-- Wheel Information -->
             <left_joint>left_joint</left_joint>
@@ -9,5 +9,5 @@
             <wheel_diameter>0.36</wheel_diameter>
             <!-- Limits -->
-            <max_wheel_torque>15</max_wheel_torque>
+            <max_wheel_torque>200</max_wheel_torque>
             <max_wheel_acceleration>10.0</max_wheel_acceleration>
             <!-- Output -->

File: install/brokk_tracked_test/share/brokk_tracked_test/urdf/brokk170_gazebo_v2.xacro (robot description, xacro)
@@ -1,33 +1,61 @@
 <?xml version="1.0" ?>
-<robot name="brokkmodel_v1" xmlns:xacro="http://www.ros.org/wiki/xacro" >
-<xacro:property name="body_color" value="Gazebo/Silver" />
-<!--Datei von Timur-->
-<gazebo reference="base_link">
-  <material>Gazebo/DarkYellow</material>
-  <mu1>0.001</mu1>
-  <mu2>0.001</mu2>
-  <self_collide>true</self_collide>
-  <gravity>true</gravity>
-</gazebo>
-<gazebo reference="imu_link">
-  <material>Gazebo/Grey</material>
-  <mu1>1</mu1>
-  <mu2>1</mu2>
-  <self_collide>false</self_collide>
-  <gravity>true</gravity>
-</gazebo>
-<gazebo reference="wheel_left_link">
-  <material>Gazebo/Grey</material>
-  <mu1>40</mu1>
-  <mu2>40</mu2>
-  <self_collide>false</self_collide>
-  <gravity>true</gravity>
-</gazebo>
-<gazebo reference="wheel_right_link">
-  <material>Gazebo/Grey</material>
-  <mu1>40</mu1>
-  <mu2>40</mu2>
-  <self_collide>false</self_collide>
-  <gravity>true</gravity>
-</gazebo>
+<robot name="brokkmodel_v2" xmlns:xacro="http://www.ros.org/wiki/xacro" >
+  <xacro:property name="body_color" value="Gazebo/Silver" />
+  <!--Datei von Timur-->
+  <gazebo reference="base_link">
+    <material>Gazebo/DarkYellow</material>
+    <mu1>0.001</mu1>
+    <mu2>0.001</mu2>
+    <self_collide>true</self_collide>
+    <gravity>true</gravity>
+  </gazebo>
+  <gazebo reference="imu_link">
+    <material>Gazebo/Grey</material>
+    <mu1>1</mu1>
+    <mu2>1</mu2>
+    <self_collide>false</self_collide>
+    <gravity>true</gravity>
+  </gazebo>
+  <gazebo reference="wheel_left_link">
+    <material>Gazebo/Grey</material>
+    <mu1>40</mu1>
+    <mu2>40</mu2>
+    <self_collide>false</self_collide>
+    <gravity>true</gravity>
+  </gazebo>
+  <gazebo reference="wheel_right_link">
+    <material>Gazebo/Grey</material>
+    <mu1>40</mu1>
+    <mu2>40</mu2>
+    <self_collide>false</self_collide>
+    <gravity>true</gravity>
+  </gazebo>
+  <gazebo reference="right_track_behind_link">
+    <material>Gazebo/Grey</material>
+    <mu1>0.018</mu1>
+    <mu2>0.018</mu2>
+    <self_collide>true</self_collide>
+    <gravity>true</gravity>
+  </gazebo>
+  <gazebo reference="right_track_front_link">
+    <material>Gazebo/Grey</material>
+    <mu1>0.018</mu1>
+    <mu2>0.018</mu2>
+    <self_collide>true</self_collide>
+    <gravity>true</gravity>
+  </gazebo>
+  <gazebo reference="left_track_behind_link">
+    <material>Gazebo/Blue</material>
+    <mu1>0.018</mu1>
+    <mu2>0.018</mu2>
+    <self_collide>true</self_collide>
+    <gravity>true</gravity>
+  </gazebo>
+  <gazebo reference="left_track_front_link">
+    <material>Gazebo/Blue</material>
+    <mu1>0.018</mu1>
+    <mu2>0.018</mu2>
+    <self_collide>true</self_collide>
+    <gravity>true</gravity>
+  </gazebo>
 </robot>

File: install/brokk_tracked_test/share/brokk_tracked_test/urdf/brokkmodel_v2.xacro (robot description, xacro)
@@ -49,7 +49,18 @@
   <xacro:property name="brokk_arm_vel_limit" value="50.0"/>
   <xacro:property name="k_velocity" value="1.0"/>
-  <xacro:property name="wheel_mass" value="50"/>
+<!--Inertia Details for the Wheel-->
+  <xacro:property name="wheel_mass" value="100"/>
   <xacro:property name="wheel_radius" value="0.18"/>
   <xacro:property name="wheel_length" value="0.18"/>
+<!-- Inertia Details for the Base-->
+  <xacro:property name="base_mass" value="1400"/>
+  <xacro:property name="base_length" value="1.66"/>
+  <xacro:property name="base_width" value="0.52"/>
+  <xacro:property name="base_height" value="0.5"/>
+<!-- Inertia Details for the Boxes, that should resemble the tracks-->
+  <xacro:property name="track_mass" value="50"/>
+  <xacro:property name="track_halflength" value="0.6"/>
+  <xacro:property name="track_width" value="0.2"/>
+  <xacro:property name="track_height" value="0.36"/>
   <link name="base_footprint"/>
   <joint name="base_joint" type="fixed">
@@ -79,9 +90,12 @@
       <inertia ixx="10.0" ixy="0.0" ixz="0.0" iyy="10.0" iyz="0.0" izz="10.0" />
     </inertial> -->
-  <inertial>
-    <origin xyz="-0.08085119432482685 1.3154078217780807e-06 0.3253779518398226" rpy="0 0 0"/>
-    <mass value="44.608708998369"/>
+  <!-- <inertial>
+    <origin xyz="-0.0 0.0 0.0" rpy="0 0 0"/>
+    <mass value="1400"/>
     <inertia ixx="58.269687" iyy="164.008688" izz="152.367637" ixy="3.5e-05" iyz="-3.5e-05" ixz="26.151771"/>
-  </inertial>
+  </inertial> -->
+    <xacro:inertial_box mass="${base_mass}" x="${base_length}" y="${base_width}" z="${base_height}">
+      <origin xyz="0 0 0" rpy="0 0 0"/>
+    </xacro:inertial_box>
   </link>
   <link name="imu_link"/>
@@ -93,5 +107,5 @@
   <!-- Einheit-->
   <joint name="left_joint" type="continuous">
-    <origin xyz="0.70 0.4 0.17" rpy="0 0 0"/>
+    <origin xyz="0.07 0.4 0.18" rpy="0 0 0"/>
     <parent link="base_link"/>
     <child link="wheel_left_link"/>
@@ -105,5 +119,5 @@
       	<mesh filename="file://$(find brokk_tracked_test)/models/meshes/wheel.stl"/>
       </geometry>
-      <material name="dark"/>
+      <material name="blue"/>
     </visual>
     <collision>
@@ -123,5 +137,5 @@
   </link>
   <joint name="right_joint" type="continuous">
-    <origin xyz="0.70 -0.4 0.17" rpy="0 0 0"/>
+    <origin xyz="0.07 -0.4 0.18" rpy="0 0 0"/>
     <parent link="base_link"/>
     <child link="wheel_right_link"/>
@@ -146,3 +160,96 @@
       </xacro:inertial_cylinder>
   </link>
+    <!-- Einheit: KETTENAPPROXIMATION DURCH BLÖCKE __________________________________________________________________________________________-->
+  <joint name="right_track_behind_joint" type="fixed">
+    <origin xyz="-0.42 -0.4 0.18" rpy="0 0 0"/>
+    <parent link="base_link"/>
+    <child link="right_track_behind_link"/>
+  </joint>
+  <link name="right_track_behind_link">
+    <visual>
+      <origin xyz="0 0 0.0" rpy="0 0 0"/>
+      <geometry>
+      	<mesh filename="file://$(find brokk_tracked_test)/models/meshes/track_box_approx.stl"/>
+      </geometry>
+      <material name="dark"/>
+    </visual>
+    <collision>
+      <origin xyz="0 0 0.0" rpy="0 0 0"/>
+      <geometry>
+      	<mesh filename="file://$(find brokk_tracked_test)/models/meshes/track_box_approx.stl"/>
+      </geometry>
+    </collision>
+    <xacro:inertial_box mass="${track_mass}" x="${track_halflength}" y="${track_width}" z="${track_height}">
+      <origin xyz="0 0 0" rpy="0 0 0"/>
+    </xacro:inertial_box>
+  </link>
+ <joint name="right_track_front_joint" type="fixed">
+    <origin xyz="0.56 -0.4 0.18" rpy="0 0 0"/>
+    <parent link="base_link"/>
+    <child link="right_track_front_link"/>
+  </joint>
+  <link name="right_track_front_link">
+    <visual>
+      <origin xyz="0 0 0.0" rpy="0 0 0"/>
+      <geometry>
+      	<mesh filename="file://$(find brokk_tracked_test)/models/meshes/track_box_approx.stl"/>
+      </geometry>
+      <material name="dark"/>
+    </visual>
+    <collision>
+      <origin xyz="0 0 0.0" rpy="0 0 0"/>
+      <geometry>
+      	<mesh filename="file://$(find brokk_tracked_test)/models/meshes/track_box_approx.stl"/>
+      </geometry>
+    </collision>
+    <xacro:inertial_box mass="${track_mass}" x="${track_halflength}" y="${track_width}" z="${track_height}">
+      <origin xyz="0 0 0" rpy="0 0 0"/>
+    </xacro:inertial_box>
+  </link>
+  <joint name="left_track_behind_joint" type="fixed">
+    <origin xyz="-0.42 0.4 0.18" rpy="0 0 0"/>
+    <parent link="base_link"/>
+    <child link="left_track_behind_link"/>
+  </joint>
+  <link name="left_track_behind_link">
+    <visual>
+      <origin xyz="0 0 0.0" rpy="0 0 0"/>
+      <geometry>
+      	<mesh filename="file://$(find brokk_tracked_test)/models/meshes/track_box_approx.stl"/>
+      </geometry>
+      <material name="dark"/>
+    </visual>
+    <collision>
+      <origin xyz="0 0 0.0" rpy="0 0 0"/>
+      <geometry>
+      	<mesh filename="file://$(find brokk_tracked_test)/models/meshes/track_box_approx.stl"/>
+      </geometry>
+    </collision>
+    <xacro:inertial_box mass="${track_mass}" x="${track_halflength}" y="${track_width}" z="${track_height}">
+      <origin xyz="0 0 0" rpy="0 0 0"/>
+    </xacro:inertial_box>
+  </link>
+  <joint name="left_track_front_joint" type="fixed">
+    <origin xyz="0.56 0.4 0.18" rpy="0 0 0"/>
+    <parent link="base_link"/>
+    <child link="left_track_front_link"/>
+  </joint>
+  <link name="left_track_front_link">
+    <visual>
+      <origin xyz="0 0 0.0" rpy="0 0 0"/>
+      <geometry>
+      	<mesh filename="file://$(find brokk_tracked_test)/models/meshes/track_box_approx.stl"/>
+      </geometry>
+      <material name="dark"/>
+    </visual>
+    <collision>
+      <origin xyz="0 0 0.0" rpy="0 0 0"/>
+      <geometry>
+      	<mesh filename="file://$(find brokk_tracked_test)/models/meshes/track_box_approx.stl"/>
+      </geometry>
+    </collision>
+    <xacro:inertial_box mass="${track_mass}" x="${track_halflength}" y="${track_width}" z="${track_height}">
+      <origin xyz="0 0 0" rpy="0 0 0"/>
+    </xacro:inertial_box>
+  </link>
 </robot>

File: install/brokk_tracked_test/share/brokk_tracked_test/urdf/inertial_macros.xacro (robot description, xacro)
@@ -23,7 +23,4 @@
     <xacro:macro name="inertial_cylinder" params="mass length radius *origin">
         <inertial>
-            <geometry>
-      	        <mesh filename="file://$(find brokk)/models/meshes/wheel.stl"/>
-            </geometry>
             <!-- <xacro:insert_block name="origin"/> -->
             <mass value="${mass}" />
